Commit message: Add SLAM compatibility and gazebo lidar interaction

File: mouse_sim/urdf/mouse.urdf.xacro (robot description, xacro)
@@ -7,4 +7,5 @@
         <!-- Visual Representation in Sim -->
         <visual>
+            <origin xyz="0 0 0.0125" rpy="0 0 0"/>
             <geometry>
                 <box size="0.1 0.06 0.04"/>
@@ -16,4 +17,5 @@
         <!-- Collision Boundaries -->
         <collision>
+            <origin xyz="0 0 0.0125" rpy="0 0 0"/>
             <geometry>
                 <box size="0.10 0.06 0.04"/> <!-- Should be same as visual -->
@@ -30,5 +32,5 @@
         <parent link="base_footprint"/>
         <child link="base_link"/>
-        <origin xyz="0 0 0.0225" rpy="0 0 0"/>
+        <origin xyz="0 0 0.01" rpy="0 0 0"/>
     </joint>
     <!-- Wheel Link Template -->
@@ -58,5 +60,5 @@
             <parent link="base_link"/>
             <child link="${position}_wheel"/>
-            <origin xyz="${x_reflect * 0.025} ${y_reflect * 0.03625} -0.0125" rpy="-1.5708 0 0"/>
+            <origin xyz="${x_reflect * 0.025} ${y_reflect * 0.03625} 0" rpy="-1.5708 0 0"/>
             <axis xyz="0 0 1"/>
         </joint>
@@ -67,38 +69,7 @@
     <xacro:wheel position="rear_left"   x_reflect="-1" y_reflect="1" />
     <xacro:wheel position="rear_right"  x_reflect="-1" y_reflect="-1" />
-    <!-- Visual Laser Indicator -->
-    <link name="viewport">
-        <visual>
-            <geometry>
-                <cylinder radius="0.02" length="0.015"/>
-            </geometry>
-            <material name="grey">
-                <color rgba="0.663 0.533 0.6 0.8"/>
-            </material>
-        </visual>
-    </link>
-    <link name="laser">
-        <visual>
-            <geometry>
-                <cylinder radius="0.0005" length="0.03"/>
-            </geometry>
-            <material name="magenta">
-                <color rgba="0.197 0 0.47 0.8"/>
-            </material>
-        </visual>
-    </link>
-    <!-- Laser Location -->
-    <joint name="viewport_joint" type="fixed">
-        <parent link="base_link"/>
-        <child link="viewport"/>
-        <origin xyz="-0.03 0 0.02" rpy="0 0 0"/>
-    </joint>
-    <joint name="laser_joint" type="fixed">
-        <parent link="viewport"/>
-        <child link="laser"/>
-        <origin xyz="0.01 0 0.0075" rpy="0 1.5708 0"/>
-    </joint>
     <!-- Gazebo Simulation Logic -->
     <gazebo>
+        <!-- Enable Differential Drive -->
         <plugin filename="ignition-gazebo-diff-drive-system" name="ignition::gazebo::systems::DiffDrive">
             <!-- Wheel Joints -->
@@ -108,5 +79,5 @@
             <right_joint>rear_right_wheel_joint</right_joint>
             <!-- Kinematics -->
-            <wheel_separation>0.725</wheel_separation>
+            <wheel_separation>0.0725</wheel_separation>
             <wheel_radius>0.01</wheel_radius>
             <!-- Limits -->
@@ -120,3 +91,5 @@
         </plugin>
     </gazebo>
+    <!-- File Inclusions -->
+    <xacro:include filename="lidar.xacro" /> <!-- Includes Lidar Capabilities -->
 </robot>

File: mouse_sim/worlds/empty_macro.sdf.xacro (robot description, xacro)
@@ -11,4 +11,7 @@
 		<plugin filename="gz-sim-user-commands-system" name="gz::sim::systems::UserCommands"/>
 		<plugin filename="gz-sim-scene-broadcaster-system" name="gz::sim::systems::SceneBroadcaster"/>
+		<plugin filename="ignition-gazebo-sensors-system" name="ignition::gazebo::systems::Sensors">
+			<render_engine>ogre2</render_engine>
+		</plugin>
 		<!-- Light Source (Needed or it'll be pitch black)-->
 		<light type="directional" name="sun">
